Commit message: Updated URDF geometries, added RViz launch file and config.

File: description/urdf/base.xacro (robot description, xacro)
@@ -1,22 +1,29 @@
-<xacro:macro name="base_link" params="">
-  <link name="base_link">
-    <visual>
-      <geometry>
-        <box size="0.25 0.20 0.05"/>
-      </geometry>
-      <material name="gray">
-        <color rgba="0.5 0.5 0.5 1"/>
-      </material>
-    </visual>
-    <collision>
-      <geometry>
-        <box size="0.25 0.20 0.05"/>
-      </geometry>
-    </collision>
-    <inertial>
-      <mass value="2.0"/>
-      <inertia ixx="0.02" iyy="0.02" izz="0.03"
-               ixy="0" ixz="0" iyz="0"/>
-    </inertial>
-  </link>
-</xacro:macro>
+<?xml version="1.0"?>
+<robot xmlns:xacro="http://www.ros.org/wiki/xacro">
+  <xacro:macro name="base_link" params="">
+    <!-- Base link at wheel axle height -->
+    <link name="base_link">
+      <visual>
+        <origin xyz="0 0 0.0175"/>
+        <geometry>
+          <box size="0.20 0.095 0.065"/>
+        </geometry>
+        <material name="gray">
+          <color rgba="0.5 0.5 0.5 1"/>
+        </material>
+      </visual>
+      <collision>
+        <origin xyz="0 0 0.0175"/>
+        <geometry>
+          <box size="0.20 0.095 0.065"/>
+        </geometry>
+      </collision>
+      <inertial>
+        <mass value="2.0"/>
+        <origin xyz="0 0 0.0175"/>
+        <inertia ixx="0.02" iyy="0.02" izz="0.03"
+                 ixy="0" ixz="0" iyz="0"/>
+      </inertial>
+    </link>
+  </xacro:macro>
+</robot>

File: description/urdf/camera_gimbal.xacro (robot description, xacro)
@@ -1,25 +1,58 @@
-<xacro:macro name="camera_gimbal" params="">
-  <!-- Pan joint -->
-  <link name="gimbal_pan"/>
-  <joint name="gimbal_pan_joint" type="continuous">
-    <parent link="base_link"/>
-    <child link="gimbal_pan"/>
-    <origin xyz="0 0 0.10"/>
-    <axis xyz="0 0 1"/>
-  </joint>
-  <!-- Tilt joint -->
-  <link name="gimbal_tilt"/>
-  <joint name="gimbal_tilt_joint" type="continuous">
-    <parent link="gimbal_pan"/>
-    <child link="gimbal_tilt"/>
-    <origin xyz="0 0 0.03"/>
-    <axis xyz="0 1 0"/>
-  </joint>
-  <!-- Camera -->
-  <link name="camera_link"/>
-  <joint name="camera_joint" type="fixed">
-    <parent link="gimbal_tilt"/>
-    <child link="camera_link"/>
-    <origin xyz="0.02 0 0"/>
-  </joint>
-</xacro:macro>
+<?xml version="1.0"?>
+<robot xmlns:xacro="http://www.ros.org/wiki/xacro">
+  <xacro:macro name="camera_gimbal" params="">
+    <!-- PAN LINK -->
+    <link name="gimbal_pan">
+      <visual>
+        <origin xyz="0.04 0 0.05" rpy="0 0 0"/>
+        <geometry>
+          <cylinder radius="0.015" length="0.02"/>
+        </geometry>
+        <material name="dark_gray">
+          <color rgba="0.3 0.3 0.3 1"/>
+        </material>
+      </visual>
+    </link>
+    <joint name="gimbal_pan_joint" type="continuous">
+      <parent link="base_link"/>
+      <child link="gimbal_pan"/>
+      <origin xyz="0.04 0 0.05" rpy="0 0 0"/>
+      <axis xyz="0 0 1"/> <!-- yaw -->
+    </joint>
+    <!-- TILT LINK -->
+    <link name="gimbal_tilt">
+      <visual>
+        <origin xyz="0.04 0 0.075" rpy="0 0 0"/>
+        <geometry>
+          <cylinder radius="0.015" length="0.02"/>
+        </geometry>
+        <material name="dark_gray">
+          <color rgba="0.3 0.3 0.3 1"/>
+        </material>
+      </visual>
+    </link>
+    <joint name="gimbal_tilt_joint" type="continuous">
+      <parent link="gimbal_pan"/>
+      <child link="gimbal_tilt"/>
+      <origin xyz="0 0 0.025" rpy="0 0 0"/>
+      <axis xyz="0 1 0"/> <!-- pitch -->
+    </joint>
+    <!-- CAMERA LINK -->
+    <link name="camera_link">
+      <visual>
+        <origin xyz="0.10 0 0.075" rpy="0 0 0"/>
+        <geometry>
+          <box size="0.04 0.04 0.04"/>
+        </geometry>
+        <material name="blue">
+          <color rgba="0.2 0.2 0.8 1"/>
+        </material>
+      </visual>
+    </link>
+    <joint name="camera_joint" type="fixed">
+      <parent link="gimbal_tilt"/>
+      <child link="camera_link"/>
+      <origin xyz="0.06 0 0" rpy="0 0 0"/>
+    </joint>
+  </xacro:macro>
+</robot>

File: description/urdf/sensors.xacro (robot description, xacro)
@@ -1,23 +1,39 @@
-<xacro:macro name="sensor_mounts" params="">
-  <!-- IMU -->
-  <link name="imu_link"/>
-  <joint name="imu_joint" type="fixed">
-    <parent link="base_link"/>
-    <child link="imu_link"/>
-    <origin xyz="0 0 0.05"/>
-  </joint>
-  <!-- Ultrasonic -->
-  <link name="ultrasonic_link"/>
-  <joint name="ultrasonic_joint" type="fixed">
-    <parent link="base_link"/>
-    <child link="ultrasonic_link"/>
-    <origin xyz="0.12 0 0.03"/>
-  </joint>
-  <!-- Line follower -->
-  <link name="line_follower_link"/>
-  <joint name="line_follower_joint" type="fixed">
-    <parent link="base_link"/>
-    <child link="line_follower_link"/>
-    <origin xyz="0.10 0 -0.02"/>
-  </joint>
-</xacro:macro>
+<?xml version="1.0"?>
+<robot xmlns:xacro="http://www.ros.org/wiki/xacro">
+  <xacro:macro name="sensor_mounts" params="">
+    <!-- LINE FOLLOWER -->
+    <link name="line_follower_link">
+      <visual>
+        <origin xyz="0.10 0 -0.015" rpy="0 0 0"/>
+        <geometry>
+          <box size="0.04 0.02 0.01"/>
+        </geometry>
+        <material name="black">
+          <color rgba="0.1 0.1 0.1 1"/>
+        </material>
+      </visual>
+    </link>
+    <joint name="line_follower_joint" type="fixed">
+      <parent link="base_link"/>
+      <child link="line_follower_link"/>
+      <origin xyz="0.10 0 -0.015" rpy="0 0 0"/>
+    </joint>
+    <!-- ULTRASONIC SENSOR -->
+    <link name="ultrasonic_link">
+      <visual>
+        <origin xyz="0.08 0 0.03" rpy="0 0 0"/>
+        <geometry>
+          <box size="0.03 0.03 0.02"/>
+        </geometry>
+        <material name="silver">
+          <color rgba="0.7 0.7 0.7 1"/>
+        </material>
+      </visual>
+    </link>
+    <joint name="ultrasonic_joint" type="fixed">
+      <parent link="base_link"/>
+      <child link="ultrasonic_link"/>
+      <origin xyz="0.08 0 0.03" rpy="0 0 0"/>
+    </joint>
+  </xacro:macro>
+</robot>

File: description/urdf/wheels.xacro (robot description, xacro)
@@ -1,59 +1,97 @@
-<xacro:macro name="mecanum_wheels" params="">
-  <!-- Wheel parameters -->
-  <xacro:property name="wheel_radius" value="0.03"/>
-  <xacro:property name="wheel_width" value="0.02"/>
-  <xacro:property name="wheel_offset_x" value="0.12"/>
-  <xacro:property name="wheel_offset_y" value="0.10"/>
-  <!-- Front Right -->
-  <link name="wheel_fr">
-    <visual>
-      <geometry><cylinder radius="${wheel_radius}" length="${wheel_width}"/></geometry>
-      <origin xyz="${wheel_offset_x} -${wheel_offset_y} 0" rpy="0 1.57 0"/>
-    </visual>
-  </link>
-  <joint name="joint_wheel_fr" type="continuous">
-    <parent link="base_link"/>
-    <child link="wheel_fr"/>
-    <origin xyz="${wheel_offset_x} -${wheel_offset_y} 0"/>
-    <axis xyz="0 1 0"/>
-  </joint>
-  <!-- Front Left -->
-  <link name="wheel_fl">
-    <visual>
-      <geometry><cylinder radius="${wheel_radius}" length="${wheel_width}"/></geometry>
-      <origin xyz="${wheel_offset_x} ${wheel_offset_y} 0" rpy="0 1.57 0"/>
-    </visual>
-  </link>
-  <joint name="joint_wheel_fl" type="continuous">
-    <parent link="base_link"/>
-    <child link="wheel_fl"/>
-    <origin xyz="${wheel_offset_x} ${wheel_offset_y} 0"/>
-    <axis xyz="0 1 0"/>
-  </joint>
-  <!-- Rear Left -->
-  <link name="wheel_rl">
-    <visual>
-      <geometry><cylinder radius="${wheel_radius}" length="${wheel_width}"/></geometry>
-      <origin xyz="-${wheel_offset_x} ${wheel_offset_y} 0" rpy="0 1.57 0"/>
-    </visual>
-  </link>
-  <joint name="joint_wheel_rl" type="continuous">
-    <parent link="base_link"/>
-    <child link="wheel_rl"/>
-    <origin xyz="-${wheel_offset_x} ${wheel_offset_y} 0"/>
-    <axis xyz="0 1 0"/>
-  </joint>
-  <!-- Rear Right -->
-  <link name="wheel_rr">
-    <visual>
-      <geometry><cylinder radius="${wheel_radius}" length="${wheel_width}"/></geometry>
-      <origin xyz="-${wheel_offset_x} -${wheel_offset_y} 0" rpy="0 1.57 0"/>
-    </visual>
-  </link>
-  <joint name="joint_wheel_rr" type="continuous">
-    <parent link="base_link"/>
-    <child link="wheel_rr"/>
-    <origin xyz="-${wheel_offset_x} -${wheel_offset_y} 0"/>
-    <axis xyz="0 1 0"/>
-  </joint>
-</xacro:macro>
+<?xml version="1.0"?>
+<robot xmlns:xacro="http://www.ros.org/wiki/xacro">
+  <xacro:macro name="mecanum_wheels" params="">
+    <!-- Real geometry -->
+    <xacro:property name="wheel_radius" value="0.03"/>
+    <xacro:property name="wheel_width" value="0.03"/>
+    <xacro:property name="wheelbase" value="0.120"/>
+    <xacro:property name="track" value="0.1410"/>
+    <!-- Derived offsets -->
+    <xacro:property name="offset_x" value="${wheelbase / 2.0}"/>
+    <xacro:property name="offset_y" value="${track / 2.0}"/>
+    <!-- FRONT RIGHT -->
+    <link name="wheel_fr">
+      <visual>
+        <origin xyz="${offset_x} -${offset_y} 0" rpy="0 1.57 0"/>
+        <geometry>
+          <cylinder radius="${wheel_radius}" length="${wheel_width}"/>
+        </geometry>
+      </visual>
+      <collision>
+        <origin xyz="${offset_x} -${offset_y} 0" rpy="0 1.57 0"/>
+        <geometry>
+          <cylinder radius="${wheel_radius}" length="${wheel_width}"/>
+        </geometry>
+      </collision>
+    </link>
+    <joint name="joint_wheel_fr" type="continuous">
+      <parent link="base_link"/>
+      <child link="wheel_fr"/>
+      <origin xyz="${offset_x} -${offset_y} 0"/>
+      <axis xyz="0 1 0"/>
+    </joint>
+    <!-- FRONT LEFT -->
+    <link name="wheel_fl">
+      <visual>
+        <origin xyz="${offset_x} ${offset_y} 0" rpy="0 1.57 0"/>
+        <geometry>
+          <cylinder radius="${wheel_radius}" length="${wheel_width}"/>
+        </geometry>
+      </visual>
+      <collision>
+        <origin xyz="${offset_x} ${offset_y} 0" rpy="0 1.57 0"/>
+        <geometry>
+          <cylinder radius="${wheel_radius}" length="${wheel_width}"/>
+        </geometry>
+      </collision>
+    </link>
+    <joint name="joint_wheel_fl" type="continuous">
+      <parent link="base_link"/>
+      <child link="wheel_fl"/>
+      <origin xyz="${offset_x} ${offset_y} 0"/>
+      <axis xyz="0 1 0"/>
+    </joint>
+    <!-- REAR LEFT -->
+    <link name="wheel_rl">
+      <visual>
+        <origin xyz="-${offset_x} ${offset_y} 0" rpy="0 1.57 0"/>
+        <geometry>
+          <cylinder radius="${wheel_radius}" length="${wheel_width}"/>
+        </geometry>
+      </visual>
+      <collision>
+        <origin xyz="-${offset_x} ${offset_y} 0" rpy="0 1.57 0"/>
+        <geometry>
+          <cylinder radius="${wheel_radius}" length="${wheel_width}"/>
+        </geometry>
+      </collision>
+    </link>
+    <joint name="joint_wheel_rl" type="continuous">
+      <parent link="base_link"/>
+      <child link="wheel_rl"/>
+      <origin xyz="-${offset_x} ${offset_y} 0"/>
+      <axis xyz="0 1 0"/>
+    </joint>
+    <!-- REAR RIGHT -->
+    <link name="wheel_rr">
+      <visual>
+        <origin xyz="-${offset_x} -${offset_y} 0" rpy="0 1.57 0"/>
+        <geometry>
+          <cylinder radius="${wheel_radius}" length="${wheel_width}"/>
+        </geometry>
+      </visual>
+      <collision>
+        <origin xyz="-${offset_x} -${offset_y} 0" rpy="0 1.57 0"/>
+        <geometry>
+          <cylinder radius="${wheel_radius}" length="${wheel_width}"/>
+        </geometry>
+      </collision>
+    </link>
+    <joint name="joint_wheel_rr" type="continuous">
+      <parent link="base_link"/>
+      <child link="wheel_rr"/>
+      <origin xyz="-${offset_x} -${offset_y} 0"/>
+      <axis xyz="0 1 0"/>
+    </joint>
+  </xacro:macro>
+</robot>
