Commit message: RViz now launchs from display launch file, URDF file is working but needs updates eventually, wheels are sideways.

File: description/urdf/base.xacro (robot description, xacro)
@@ -19,10 +19,4 @@
         </geometry>
       </collision>
-      <inertial>
-        <mass value="2.0"/>
-        <origin xyz="0 0 0.0175"/>
-        <inertia ixx="0.02" iyy="0.02" izz="0.03"
-                 ixy="0" ixz="0" iyz="0"/>
-      </inertial>
     </link>
   </xacro:macro>

File: description/urdf/robot.urdf.xacro (robot description, xacro)
@@ -1,13 +1,13 @@
 <?xml version="1.0"?>
-<robot name="mecanum_bot" xmlns:xacro="http://www.ros.org/wiki/xacro">
+<robot name="turbopi" xmlns:xacro="http://www.ros.org/wiki/xacro">
   <!-- Include modular components -->
-  <xacro:include filename="$(find description)/urdf/base.xacro"/>
-  <xacro:include filename="$(find description)/urdf/wheels.xacro"/>
-  <xacro:include filename="$(find description)/urdf/sensors.xacro"/>
-  <xacro:include filename="$(find description)/urdf/camera_gimbal.xacro"/>
+  <xacro:include filename="base.xacro"/>
+  <xacro:include filename="wheels.xacro"/>
+  <xacro:include filename="sensors.xacro"/>
+  <xacro:include filename="camera_gimbal.xacro"/>
   <!-- Instantiate components -->
-  <base_link/>
-  <mecanum_wheels/>
-  <sensor_mounts/>
-  <camera_gimbal/>
+  <xacro:base_link/>
+  <xacro:mecanum_wheels/>
+  <xacro:sensor_mounts/>
+  <xacro:camera_gimbal/>
 </robot>
